File: USBC_UART_Dock_Prototype/USBC_UART_Dock_Prototype.kicad_pcb (KiCad board)
At the start: 2 copper layers, 0 parts

Commit message: Rev. A ready for review
Parts:
- added C1: 47p, Capacitor_SMD:C_1206_3216Metric_Pad1.33x1.80mm_HandSolder, F.Cu at (121.5, 86.0)
- added C10: 1u, Capacitor_SMD:C_1206_3216Metric_Pad1.33x1.80mm_HandSolder, F.Cu at (158.4, 90.1)
- added C11: 0.1u, Capacitor_SMD:C_0603_1608Metric_Pad1.08x0.95mm_HandSolder, F.Cu at (163.4, 88.0)
- added C12: 10u, Capacitor_SMD:C_1206_3216Metric_Pad1.33x1.80mm_HandSolder, F.Cu at (160.3, 84.1)
- added C13: 0.1u, Capacitor_SMD:C_0603_1608Metric_Pad1.08x0.95mm_HandSolder, F.Cu at (134.5, 100.1)
- added C16: 1u, Capacitor_SMD:C_1206_3216Metric_Pad1.33x1.80mm_HandSolder, F.Cu at (121.7, 82.8)
- added C17: 1u, Capacitor_SMD:C_1206_3216Metric_Pad1.33x1.80mm_HandSolder, F.Cu at (132.7, 85.4)
- added C2: 47u, Capacitor_SMD:C_1206_3216Metric_Pad1.33x1.80mm_HandSolder, F.Cu at (141.9, 80.5)
- added C3: 47p, Capacitor_SMD:C_1206_3216Metric_Pad1.33x1.80mm_HandSolder, F.Cu at (121.4, 102.0)
- added C4: 47u, Capacitor_SMD:C_1206_3216Metric_Pad1.33x1.80mm_HandSolder, F.Cu at (135.2, 80.5)
- added C5: 47u, Capacitor_SMD:C_1206_3216Metric_Pad1.33x1.80mm_HandSolder, F.Cu at (131.8, 80.5)
- added C6: 0.1u, Capacitor_SMD:C_0603_1608Metric_Pad1.08x0.95mm_HandSolder, F.Cu at (128.2, 90.2)
- added C7: 0.1u, Capacitor_SMD:C_0603_1608Metric_Pad1.08x0.95mm_HandSolder, F.Cu at (145.4, 84.2)
- added C8: 47p, Capacitor_SMD:C_1206_3216Metric_Pad1.33x1.80mm_HandSolder, F.Cu at (149.7, 92.5)
- added C9: 47p, Capacitor_SMD:C_1206_3216Metric_Pad1.33x1.80mm_HandSolder, F.Cu at (149.8, 97.5)
- added D1: LED_GREEN, LED_SMD:LED_0805_2012Metric_Pad1.15x1.40mm_HandSolder, F.Cu at (148.2, 77.5)
- added D2: LED_GREEN, LED_SMD:LED_0805_2012Metric_Pad1.15x1.40mm_HandSolder, F.Cu at (151.6, 77.5)
- added D3: LED_GREEN, LED_SMD:LED_0805_2012Metric_Pad1.15x1.40mm_HandSolder, F.Cu at (155.0, 77.5)
- added D4: LED_RED, LED_SMD:LED_0805_2012Metric_Pad1.15x1.40mm_HandSolder, F.Cu at (158.4, 77.5)
- added D5: LED_RED, LED_SMD:LED_0805_2012Metric_Pad1.15x1.40mm_HandSolder, F.Cu at (161.8, 77.5)
- added D6: LED_GREEN, LED_SMD:LED_0805_2012Metric_Pad1.15x1.40mm_HandSolder, F.Cu at (165.2, 77.5)
- added G***: LOGO, PROVE:PROVE-logo, F.Cu at (159.0, 102.0)
- added J1: Conn_01x01, Connector:Banana_Jack_1Pin, F.Cu at (122.5, 67.3)
- added J2: Conn_01x01, Connector:Banana_Jack_1Pin, F.Cu at (140.0, 67.3)
- added J3: Conn_01x05_Socket, Connector_PinSocket_2.54mm:PinSocket_1x05_P2.54mm_Vertical, F.Cu at (150.4, 63.4)
- added J4: USB4085-GF-A, Connector_USB:USB_C_Receptacle_GCT_USB4085, F.Cu at (162.8, 97.3)
- added R1: 100k, Resistor_SMD:R_1206_3216Metric_Pad1.30x1.75mm_HandSolder, F.Cu at (145.9, 90.1)
- added R2: 16, Resistor_SMD:R_1206_3216Metric_Pad1.30x1.75mm_HandSolder, F.Cu at (145.7, 96.2)
- added R3: 16, Resistor_SMD:R_1206_3216Metric_Pad1.30x1.75mm_HandSolder, F.Cu at (145.7, 93.8)
- added R4: 2.2k, Resistor_SMD:R_1206_3216Metric_Pad1.30x1.75mm_HandSolder, F.Cu at (148.2, 71.3)
- added R5: 2.2k, Resistor_SMD:R_1206_3216Metric_Pad1.30x1.75mm_HandSolder, F.Cu at (151.8, 71.3)
- added R6: 2.2k, Resistor_SMD:R_1206_3216Metric_Pad1.30x1.75mm_HandSolder, F.Cu at (155.4, 71.3)
- added R7: 2.2k, Resistor_SMD:R_1206_3216Metric_Pad1.30x1.75mm_HandSolder, F.Cu at (158.7, 71.3)
- added R8: 2.2k, Resistor_SMD:R_1206_3216Metric_Pad1.30x1.75mm_HandSolder, F.Cu at (161.9, 71.3)
- added R9: 2.2k, Resistor_SMD:R_1206_3216Metric_Pad1.30x1.75mm_HandSolder, F.Cu at (165.6, 71.3)
- added U1: FT312D, Package_QFP:LQFP-32_7x7mm_P0.8mm, F.Cu at (135.4, 92.6)
- added U2: TPS25810, PROVE:WQFN-20-3x4mm, F.Cu at (148.7, 85.6)
- added U3: TPD6S300A, Package_DFN_QFN:WQFN-20-1EP_3x3mm_P0.4mm_EP1.7x1.7mm_ThermalVias, F.Cu at (158.2, 93.7)
- added U5: LP5907MFX-3.3/NOPB, Package_TO_SOT_SMD:SOT-23-5_HandSoldering, F.Cu at (127.5, 84.3)
- added Y1: 12 MHz, Crystal:Crystal_SMD_HC49-SD, F.Cu at (123.0, 94.0)
Routing:
- net /nUSB_ERROR: track 0.00 -> 44.3 mm, vias 0 -> 2
- net /TX_ACTIVE: track 0.00 -> 37.4 mm, vias 0 -> 2
- net /RTS: track 0.00 -> 35.8 mm, vias 0 -> 1
- net /UART_TX: track 0.00 -> 35.2 mm, vias 0 -> 1
- net /CTS: track 0.00 -> 34.7 mm, vias 0 -> 1
- net /UART_RX: track 0.00 -> 33.3 mm, vias 0 -> 1
- net /nPWR_FLT: track 0.00 -> 32.0 mm
- net +3.3V: track 0.00 -> 25.7 mm, vias 0 -> 23
- net GND: track 0.00 -> 23.7 mm, vias 0 -> 17
- net /XTOUT: track 0.00 -> 15.4 mm
- net /XTIN: track 0.00 -> 13.0 mm
- net /CONN_USB_CC2: track 0.00 -> 12.3 mm
- net /USB_D-: track 0.00 -> 10.3 mm
- net /USB_D+: track 0.00 -> 10.2 mm
- net /USB_CC1: track 0.00 -> 9.92 mm
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- added copper zone on F.Cu, net +3.3V
- added copper zone on In2.Cu, net +3.3V
- added copper zone on F.Cu, net +5V
- added copper zone on F.Cu, net +VUSB
- added copper zone on In2.Cu, net +VUSB
- added copper zone on B.Cu, net GND
- added copper zone on F.Cu, net GND
- added copper zone on In1.Cu, net GND
Other:
- board outline added: 54.1 x 45.5 mm
- copper layers 2 -> 4
- board text added: "+5V"
- board text added: "CTS"
- board text added: "GND"
- board text added: "LD_DET"
- board text added: "POL"
- board text added: "PWR_FLT"
- board text added: "RTS"
- board text added: "RX"
- board text added: "TX"
- board text added: "TX_ACTIVE"
- board text added: "UFP"
- board text added: "USB-C UART Dock Prototype - Rev. A Designer: Lin Knudsen Date: 10/20/2024"
- board text added: "USB_ERR"
