File: USBC_UART_Dock_Prototype/USBC_UART_Dock_Prototype.kicad_sch (KiCad schematic)
At the start: 38 parts, among them J1 Conn_01x01, J2 Conn_01x01, J3 Conn_01x05_Socket, J4 USB4085-GF-A, U1 FT312D, U2 TPS25810, U3 TPD6S300A, U5 LP5907MFX-3.3/NOPB, Y1 12 MHz

Commit message: Rev. A ready for review
Parts:
- removed R2, R3: 27, Resistor_SMD:R_1206_3216Metric_Pad1.30x1.75mm_HandSolder, symbol PROVE:RT1206BRD0727RL
- added C13: 0.1u, Capacitor_SMD:C_0603_1608Metric_Pad1.08x0.95mm_HandSolder, symbol PROVE:GRM188R72A104KA35D
- added R2, R3: 16, Resistor_SMD:R_1206_3216Metric_Pad1.30x1.75mm_HandSolder, symbol PROVE:RC1206FR-0716RL
- C11, C6, C7: symbol PROVE:GRM188R71H104KA93D -> PROVE:GRM188R72A104KA35D
- J1, J2, J3: now left out of the parts list
Connections:
- net +3.3V: now also C13.1
- net CONN_USB_D+: now also U3.1 (C_SBU1); no longer U3.2 (C_SBU2)
- net CONN_USB_D-: now also U3.2 (C_SBU2); no longer U3.1 (C_SBU1)
- net GND: now also C13.2
- net USB_D+: now also U3.15 (SBU1), R2.2; no longer U3.14 (SBU2)
- net USB_D-: now also U3.14 (SBU2), R3.2; no longer U3.15 (SBU1)
- net +VUSB: now reaches C12.1, J4.A4 (VBUS), J4.A9 (VBUS), J4.B4 (VBUS), J4.B9 (VBUS), U2.14 (OUT), U2.15 (OUT)
- net FT_USB_D-: now reaches U1.18 (USBDM)
- net FT_USB_D-: now also R3.1
- net +1.8 V: now reaches C6.1, U1.3 (AVCC), U1.7 (VREGOUT)
- net XTIN: now reaches C1.1, U1.4 (XTIN), Y1.1
- net XTOUT: now reaches C3.1, U1.5 (XTOUT), Y1.2
- net FT_USB_D+: now reaches U1.17 (USBDP)
- net FT_USB_D+: now also R2.1
Other:
- company: PROVE Lab -> (none)
