File: Basic_Node_Board/Basic_Node_Board.kicad_pcb (KiCad board)
At the start: 2 copper layers, 0 parts

Commit message: Initial PCB design for sensor board
Parts:
- added C1: 0.1u, Capacitor_SMD:C_1206_3216Metric_Pad1.33x1.80mm_HandSolder, F.Cu at (70.0, 100.6)
- added C2: 30p, Capacitor_SMD:C_1206_3216Metric_Pad1.33x1.80mm_HandSolder, F.Cu at (70.0, 106.4)
- added C3: 30p, Capacitor_SMD:C_1206_3216Metric_Pad1.33x1.80mm_HandSolder, F.Cu at (92.9, 111.5)
- added C4: 2.2u, Capacitor_SMD:CP_Elec_4x5.4, F.Cu at (110.7, 125.0)
- added C5: 0.1u, Capacitor_SMD:C_1206_3216Metric_Pad1.33x1.80mm_HandSolder, F.Cu at (99.4, 111.5)
- added C6: 10u, Capacitor_SMD:C_1206_3216Metric_Pad1.33x1.80mm_HandSolder, F.Cu at (118.0, 125.1)
- added C7: 10u, Capacitor_SMD:C_1206_3216Metric_Pad1.33x1.80mm_HandSolder, F.Cu at (118.2, 121.1)
- added J1: Conn_01x02_Pin, TerminalBlock_TE-Connectivity:TerminalBlock_TE_282834-2_1x02_P2.54mm_Horizontal, F.Cu at (70.0, 116.0)
- added J2: Conn_01x02, TerminalBlock_TE-Connectivity:TerminalBlock_TE_282834-2_1x02_P2.54mm_Horizontal, F.Cu at (79.0, 124.5)
- added J3: Conn_01x19_Socket, Connector_PinHeader_1.00mm:PinHeader_1x19_P1.00mm_Vertical, F.Cu at (109.5, 73.5)
- added J5: Conn_01x19_Socket, Connector_PinHeader_1.00mm:PinHeader_1x19_P1.00mm_Vertical, F.Cu at (70.0, 73.5)
- added L1: 10u, PROVE:WE-LQS_5040, F.Cu at (94.2, 124.0)
- added R1: 30m, Resistor_SMD:R_1206_3216Metric_Pad1.30x1.75mm_HandSolder, F.Cu at (115.5, 91.0)
- added R2: 0, Resistor_SMD:R_1206_3216Metric_Pad1.30x1.75mm_HandSolder, F.Cu at (74.5, 111.5)
- added R3: 0, Resistor_SMD:R_1206_3216Metric_Pad1.30x1.75mm_HandSolder, F.Cu at (86.5, 111.5)
- added R4: 120, Resistor_SMD:R_1206_3216Metric_Pad1.30x1.75mm_HandSolder, F.Cu at (80.5, 111.5)
- added R5: 115k, Resistor_SMD:R_1206_3216Metric_Pad1.30x1.75mm_HandSolder, F.Cu at (102.0, 118.0)
- added R6: 22.1k, Resistor_SMD:R_1206_3216Metric_Pad1.30x1.75mm_HandSolder, F.Cu at (96.0, 118.0)
- added U1: INA220 Current Monitor, PROVE:DGS10, F.Cu at (109.0, 114.5)
- added U2: ESP32-DEVKIT-C, PROVE:MODULE_ESP32-DEVKITC, F.Cu at (89.8, 82.5)
- added U3: TJA1050T/CM,118, Package_SO:SOIC-8_3.9x4.9mm_P1.27mm, F.Cu at (115.5, 85.5)
- added U6: AP64060WU-7, Package_TO_SOT_SMD:TSOT-23-6, F.Cu at (102.9, 124.0)
Routing:
- net Net-(U3-CANH): track 0.00 -> 105.4 mm
- net GND: track 0.00 -> 101.5 mm, vias 0 -> 4
- net +5VD: track 0.00 -> 91.8 mm
- net Net-(U3-CANL): track 0.00 -> 75.7 mm
- net +5V: track 0.00 -> 40.5 mm
- net /Microcontroller/BUCK_5V: track 0.00 -> 36.4 mm
- net /Power_Supply/12V_IN: track 0.00 -> 33.9 mm, vias 0 -> 2
- net /Microcontroller/CANL: track 0.00 -> 25.4 mm, vias 0 -> 2
- net Net-(U6-BST): track 0.00 -> 22.2 mm, vias 0 -> 2
- net Net-(U6-SW): track 0.00 -> 20.4 mm, vias 0 -> 2
- net Net-(U6-FB): track 0.00 -> 18.5 mm, vias 0 -> 2
- net Net-(J5-Pin_1): track 0.00 -> 16.8 mm
- net Net-(J3-Pin_1): track 0.00 -> 16.8 mm
- net Net-(J3-Pin_19): track 0.00 -> 16.7 mm
- net Net-(J3-Pin_2): track 0.00 -> 16.3 mm
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- added copper zone on B.Cu, net GND
Other:
- board outline added: 62.5 x 82.5 mm
