File: Basic_Node_Board/Basic_Node_Board.kicad_pcb (KiCad board)
At the start: 2 copper layers, 0 parts

Commit message: Add files via upload
Parts:
- added C1: 0.1u, Capacitor_SMD:C_1206_3216Metric_Pad1.33x1.80mm_HandSolder, F.Cu at (67.0, 122.9)
- added C2: 30p, Capacitor_SMD:C_1206_3216Metric_Pad1.33x1.80mm_HandSolder, F.Cu at (112.7, 101.5)
- added C3: 30p, Capacitor_SMD:C_1206_3216Metric_Pad1.33x1.80mm_HandSolder, F.Cu at (118.2, 110.0)
- added C4: 2.2u, Capacitor_SMD:CP_Elec_4x5.4, F.Cu at (85.5, 57.5)
- added C5: 0.1u, Capacitor_SMD:C_1206_3216Metric_Pad1.33x1.80mm_HandSolder, F.Cu at (96.8, 71.0)
- added C6: 10u, Capacitor_SMD:C_1206_3216Metric_Pad1.33x1.80mm_HandSolder, F.Cu at (78.2, 57.4)
- added C7: 10u, Capacitor_SMD:C_1206_3216Metric_Pad1.33x1.80mm_HandSolder, F.Cu at (78.1, 61.4)
- added G***: LOGO, PROVE:BAC-logo, F.Cu at (118.5, 81.5)
- added G***: LOGO, PROVE:PROVE-logo, F.Cu at (114.5, 78.5)
- added J1: Conn_01x02_Pin, TerminalBlock_TE-Connectivity:TerminalBlock_TE_282834-2_1x02_P2.54mm_Horizontal, F.Cu at (120.2, 101.2)
- added J2: Conn_01x02, TerminalBlock_TE-Connectivity:TerminalBlock_TE_282834-2_1x02_P2.54mm_Horizontal, F.Cu at (110.5, 57.0)
- added J3: Conn_01x19_Socket, Connector_PinHeader_1.00mm:PinHeader_1x19_P1.00mm_Vertical, F.Cu at (106.9, 97.9)
- added J5: Conn_01x19_Socket, Connector_PinHeader_1.00mm:PinHeader_1x19_P1.00mm_Vertical, F.Cu at (67.4, 97.9)
- added L1: 10u, PROVE:WE-LQS_5040, F.Cu at (102.0, 58.5)
- added R1: 30m, Resistor_SMD:R_1206_3216Metric_Pad1.30x1.75mm_HandSolder, F.Cu at (114.2, 126.5)
- added R2: 0, Resistor_SMD:R_1206_3216Metric_Pad1.30x1.75mm_HandSolder, F.Cu at (112.7, 105.5)
- added R3: 0, Resistor_SMD:R_1206_3216Metric_Pad1.30x1.75mm_HandSolder, F.Cu at (121.8, 110.0)
- added R4: 120, Resistor_SMD:R_1206_3216Metric_Pad1.30x1.75mm_HandSolder, F.Cu at (120.2, 116.0)
- added R5: 115k, Resistor_SMD:R_1206_3216Metric_Pad1.30x1.75mm_HandSolder, F.Cu at (94.2, 64.5)
- added R6: 22.1k, Resistor_SMD:R_1206_3216Metric_Pad1.30x1.75mm_HandSolder, F.Cu at (100.2, 64.5)
- added U1: INA220 Current Monitor, PROVE:DGS10, F.Cu at (87.2, 68.0)
- added U2: ESP32-DEVKIT-C, PROVE:MODULE_ESP32-DEVKITC, F.Cu at (87.2, 106.9)
- added U3: TJA1050T/CM,118, Package_SO:SOIC-8_3.9x4.9mm_P1.27mm, F.Cu at (114.2, 121.0)
- added U6: AP64060WU-7, Package_TO_SOT_SMD:TSOT-23-6, F.Cu at (93.4, 58.5)
Routing:
- net +5VD: track 0.00 -> 134.2 mm, vias 0 -> 2
- net GND: track 0.00 -> 43.8 mm, vias 0 -> 9
- net /Microcontroller/BUCK_5V: track 0.00 -> 36.4 mm
- net /Power_Supply/12V_IN: track 0.00 -> 26.7 mm, vias 0 -> 2
- net Net-(J3-Pin_12): track 0.00 -> 25.1 mm
- net Net-(U6-BST): track 0.00 -> 22.2 mm, vias 0 -> 2
- net Net-(J3-Pin_11): track 0.00 -> 21.3 mm
- net Net-(U6-SW): track 0.00 -> 20.4 mm, vias 0 -> 2
- net Net-(U3-CANH): track 0.00 -> 19.3 mm
- net Net-(U6-FB): track 0.00 -> 18.5 mm, vias 0 -> 2
- net Net-(J5-Pin_1): track 0.00 -> 16.8 mm
- net Net-(J3-Pin_1): track 0.00 -> 16.8 mm
- net Net-(J3-Pin_19): track 0.00 -> 16.7 mm
- net Net-(J3-Pin_2): track 0.00 -> 16.3 mm
- net Net-(J5-Pin_2): track 0.00 -> 15.7 mm
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- added copper zone on F.Cu, net +5V
- added copper zone on B.Cu, net GND
Other:
- board outline added: 62.5 x 82.5 mm
- board text added: "12V"
- board text added: "CANH"
- board text added: "CANL"
- board text added: "GND"
- board text added: "Owen Vance Jorge Garcia"
