File: Basic_Node_Board/Basic_Node_Board.kicad_pcb (KiCad board)
At the start: 2 copper layers, 0 parts

Commit message: made fixes to the buck converter
Parts:
- added C1: 0.1u, Capacitor_SMD:C_1206_3216Metric_Pad1.33x1.80mm_HandSolder, F.Cu at (121.5, 122.9)
- added C1: 0.1u, Capacitor_SMD:C_1206_3216Metric_Pad1.33x1.80mm_HandSolder, F.Cu at (155.9, 55.0)
- added C2: 30p, Capacitor_SMD:C_1206_3216Metric_Pad1.33x1.80mm_HandSolder, F.Cu at (167.2, 101.5)
- added C2: 30p, Capacitor_SMD:C_1206_3216Metric_Pad1.33x1.80mm_HandSolder, F.Cu at (153.0, 65.6)
- added C3: 30p, Capacitor_SMD:C_1206_3216Metric_Pad1.33x1.80mm_HandSolder, F.Cu at (172.8, 110.0)
- added C3: 30p, Capacitor_SMD:C_1206_3216Metric_Pad1.33x1.80mm_HandSolder, F.Cu at (156.5, 65.6)
- added C4: GRM31CR71H475KA12L, PROVE-footprints:G-31_MUR, F.Cu at (132.6, 54.5)
- added C5: C0805C122J5GACTU, PROVE-footprints:CAPC220145_88N_KEM, F.Cu at (132.7, 57.0)
- added C6: CL05C110JB5NNNC, PROVE-footprints:CAP_CL05_SAM, F.Cu at (136.0, 60.5)
- added C8: 08053C104KAT2A, PROVE-footprints:CAPC2012X94N, F.Cu at (145.8, 51.0)
- added CR1: B560C-13-F, PROVE-footprints:SMC_DIO, F.Cu at (164.5, 69.1)
- added G***: LOGO, PROVE:BAC-logo, F.Cu at (173.0, 81.5)
- added G***: LOGO, PROVE:PROVE-logo, F.Cu at (169.0, 78.5)
- added J1: Conn_01x02_Pin, TerminalBlock_TE-Connectivity:TerminalBlock_TE_282834-2_1x02_P2.54mm_Horizontal, F.Cu at (174.8, 101.2)
- added J2: Conn_01x02, TerminalBlock_TE-Connectivity:TerminalBlock_TE_282834-2_1x02_P2.54mm_Horizontal, F.Cu at (165.0, 57.0)
- added J3: Conn_01x19_Socket, Connector_PinHeader_1.00mm:PinHeader_1x19_P1.00mm_Vertical, F.Cu at (161.4, 97.9)
- added J5: Conn_01x19_Socket, Connector_PinHeader_1.00mm:PinHeader_1x19_P1.00mm_Vertical, F.Cu at (121.9, 97.9)
- added L1: SRN8040-100M, PROVE-footprints:IND_BOURNS_SRN8040, F.Cu at (174.5, 68.4)
- added R1: 30m, Resistor_SMD:R_1206_3216Metric_Pad1.30x1.75mm_HandSolder, F.Cu at (168.7, 126.5)
- added R2: 0, Resistor_SMD:R_1206_3216Metric_Pad1.30x1.75mm_HandSolder, F.Cu at (167.2, 105.5)
- added R3: 0, Resistor_SMD:R_1206_3216Metric_Pad1.30x1.75mm_HandSolder, F.Cu at (176.2, 110.0)
- added R4: 120, Resistor_SMD:R_1206_3216Metric_Pad1.30x1.75mm_HandSolder, F.Cu at (174.7, 116.0)
- added R5: RC0201FR-0723K7L, PROVE-footprints:RES_RC0201_YAG, F.Cu at (138.7, 60.2)
- added R6: CRCW0402118KFKED, PROVE-footprints:RES_CRCW_0402, F.Cu at (138.5, 58.0)
- added R7: CRCW040261K9FKED, PROVE-footprints:RES_CRCW_0402, F.Cu at (149.0, 61.5)
- added R8: CRCW040211K0FKED, PROVE-footprints:RES_CRCW_0402, F.Cu at (149.0, 60.0)
- added U1: INA220 Current Monitor, PROVE:DGS10, F.Cu at (141.7, 68.0)
- added U2: ESP32-DEVKIT-C, PROVE:MODULE_ESP32-DEVKITC, F.Cu at (141.7, 106.9)
- added U3: TJA1050T/CM,118, Package_SO:SOIC-8_3.9x4.9mm_P1.27mm, F.Cu at (168.8, 121.0)
- added U6: TPS54560BQDDARQ1, PROVE-footprints:TPS54560BQDDARQ1, F.Cu at (145.5, 55.5)
Routing:
- net +5VD: track 0.00 -> 134.2 mm, vias 0 -> 2
- net GND: track 0.00 -> 29.6 mm, vias 0 -> 6
- net Net-(J3-Pin_12): track 0.00 -> 25.1 mm
- net Net-(J3-Pin_11): track 0.00 -> 21.3 mm
- net Net-(U3-CANH): track 0.00 -> 19.3 mm
- net Net-(J5-Pin_1): track 0.00 -> 16.8 mm
- net Net-(J3-Pin_1): track 0.00 -> 16.8 mm
- net Net-(J3-Pin_19): track 0.00 -> 16.7 mm
- net Net-(J3-Pin_2): track 0.00 -> 16.3 mm
- net Net-(J5-Pin_2): track 0.00 -> 15.7 mm
- net Net-(J5-Pin_18): track 0.00 -> 15.6 mm
- net Net-(J3-Pin_3): track 0.00 -> 15.3 mm
- net Net-(J3-Pin_18): track 0.00 -> 15.2 mm
- net Net-(J3-Pin_4): track 0.00 -> 14.4 mm
- net Net-(J5-Pin_3): track 0.00 -> 14.1 mm
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- added copper zone on F.Cu, net +5V
- added copper zone on B.Cu, net GND
Other:
- board outline added: 62.5 x 82.5 mm
- board text added: "12V"
- board text added: "CANH"
- board text added: "CANL"
- board text added: "GND"
- board text added: "Owen Vance Jorge Garcia"
