File: Basic_Node_Board/Microcontroller.kicad_sch (KiCad schematic)
At the start: 11 parts, among them J1 Conn_01x02_Pin, J3 Conn_01x19_Socket, J5 Conn_01x19_Socket, U2 ESP32-DEVKIT-C, U3 TJA1050T/CM,118

Commit message: mh_initial_node_board_edits
Connections:
- net +5V: now also J5.19 (Pin_19), U2.19 (EXT_5V)
- net GND: now also J5.14 (Pin_14), U2.14 (GND1)
Changed lines of the file:
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@@
+	)
+	(junction
+		(at 118.11 93.98)
+		(diameter 0)
+		(color 0 0 0 0)
 	)
 	(junction
@@
 	)
 	(junction
+		(at 118.11 106.68)
+		(diameter 0)
+		(color 0 0 0 0)
+	)
+	(junction
 		(at 245.11 95.25)
 		(diameter 0)
@@
 	(wire
 		(pts
+			(xy 93.98 107.95) (xy 93.98 106.68)
+		)
+		(stroke
+			(width 0)
+			(type default)
+		)
+	)
+	(wire
+		(pts
+			(xy 118.11 107.95) (xy 118.11 106.68)
+		)
+		(stroke
+			(width 0)
+			(type default)
+		)
+	)
+	(wire
+		(pts
 			(xy 223.52 77.47) (xy 223.52 82.55)
 		)
@@
 	(wire
 		(pts
+			(xy 91.44 95.25) (xy 118.11 95.25)
+		)
+		(stroke
+			(width 0)
+			(type default)
+		)
+	)
+	(wire
+		(pts
 			(xy 118.11 81.28) (xy 120.65 81.28)
 		)
@@
 	(wire
 		(pts
+			(xy 118.11 95.25) (xy 118.11 93.98)
+		)
+		(stroke
+			(width 0)
+			(type default)
+		)
+	)
+	(wire
+		(pts
 			(xy 186.69 48.26) (xy 186.69 64.77)
 		)
@@
 	(wire
 		(pts
+			(xy 93.98 107.95) (xy 118.11 107.95)
+		)
+		(stroke
+			(width 0)
+			(type default)
+		)
+	)
+	(wire
+		(pts
 			(xy 118.11 86.36) (xy 120.65 86.36)
 		)
@@
 	)
 	(label "BUCK_5V"
-		(at 86.36 116.84 0)
+		(at 101.6 107.95 0)
 		(fields_autoplaced yes)
 		(effects
@@
 		)
 	)
+	(label "BUCK_GND"
+		(at 97.79 95.25 0)
+		(fields_autoplaced yes)
+		(effects
+			(font
+				(size 1.27 1.27)
+			)
+			(justify left bottom)
+		)
+	)
 	(symbol
 		(lib_id "power:GND")
-		(at 91.44 93.98 0)
+		(at 91.44 95.25 0)
 		(unit 1)
 		(exclude_from_sim no)
@@
 		(fields_autoplaced yes)
 		(property "Reference" "#PWR011"
+			(at 91.44 101.6 0)
+			(effects
+				(font
+					(size 1.27 1.27)
+				)
+				(hide yes)
+			)
+		)
+		(property "Value" "GND"
 			(at 91.44 100.33 0)
 			(effects
@@
 					(size 1.27 1.27)
 				)
-				(hide yes)
-			)
-		)
-		(property "Value" "GND"
-			(at 91.44 99.06 0)
-			(effects
-				(font
-					(size 1.27 1.27)
-				)
 			)
 		)
 		(property "Footprint" ""
-			(at 91.44 93.98 0)
+			(at 91.44 95.25 0)
 			(effects
 				(font
@@
 		)
 		(property "Datasheet" ""
-			(at 91.44 93.98 0)
+			(at 91.44 95.25 0)
 			(effects
 				(font
@@
 		)
 		(property "Description" "Power symbol creates a global label with name \"GND\" , ground"
-			(at 91.44 93.98 0)
+			(at 91.44 95.25 0)
 			(effects
 				(font
@@
 	(symbol
 		(lib_id "power:+5V")
-		(at 93.98 106.68 90)
+		(at 93.98 106.68 0)
 		(unit 1)
 		(exclude_from_sim no)
@@
 		(fields_autoplaced yes)
 		(property "Reference" "#PWR09"
-			(at 97.79 106.68 0)
+			(at 93.98 110.49 0)
 			(effects
 				(font
@@
 		)
 		(property "Value" "+5V"
-			(at 90.17 106.6799 90)
+			(at 96.52 105.4099 0)
 			(effects
 				(font
@@
 		(dnp no)
 		(property "Reference" "J1"
-			(at 267.462 77.47 0)
+			(at 258.572 73.66 0)
 			(effects
 				(font
@@
 		)
 		(property "Value" "Conn_01x02_Pin"
-			(at 268.732 75.692 0)
-			(effects
-				(font
+			(at 258.318 71.374 0)
+			(effects
+				(font

Commit message: Update Microcontroller.kicad_sch
Parts:
- added C5: 2.2u, Capacitor_SMD:CP_Elec_4x5.4, symbol PROVE:EEE-1VA2R2NR
- added C6, C7: 10u, Capacitor_SMD:C_1206_3216Metric_Pad1.33x1.80mm_HandSolder, symbol PROVE:CL31A106KPHNNNE
- added D1: BPX65, Package_TO_SOT_THT:TO-18-2_Lens, symbol Sensor_Optical:BPX65
- added L1: 10u, PROVE:WE-LQS_5040, symbol PROVE:74404054100
- added R5: 115k, Resistor_SMD:R_1206_3216Metric_Pad1.30x1.75mm_HandSolder, symbol PROVE:RC1206FR-07115KL
- added R6: 22.1k, Resistor_SMD:R_1206_3216Metric_Pad1.30x1.75mm_HandSolder, symbol PROVE:RNCP1206FTD22K1
- added U4, U5: AP64060WU-7, Package_TO_SOT_SMD:TSOT-23-6, symbol PROVE:AP64060WU-7
Connections:
- net GND: now also C5.2, C6.2, C7.2, R6.2
- new net: C6.1, C7.1, L1.2, R5.1
- new net: R5.2, R6.1

Commit message: Update Microcontroller.kicad_sch
Parts:
- removed D1: BPX65, Package_TO_SOT_THT:TO-18-2_Lens, symbol Sensor_Optical:BPX65
- added C4: 0.1u, Capacitor_SMD:C_1206_3216Metric_Pad1.33x1.80mm_HandSolder, symbol PROVE:1206B104K500CT
- added J2: Conn_01x02, symbol Connector_Generic:Conn_01x02
- added U6: AP64060WU-7, Package_TO_SOT_SMD:TSOT-23-6, symbol PROVE:AP64060WU-7
Connections:
- net +5V is gone; now on net BUCK_5V: C1.2, J5.19 (Pin_19), U2.19 (EXT_5V), U3.3 (VCC)
- net GND: now also J2.2 (Pin_2), U6.2 (GND)
- net BUCK_5V: now reaches C6.1, C7.1, L1.2, R5.1
- net at R5.2, R6.1: now also U6.3 (FB)
- net 12V_IN: now reaches C5.1
- net 12V_IN: now also J2.1 (Pin_1), U6.5 (VIN)
- net at L1.1: now also C4.2, U6.6 (SW)
- new net: C4.1, U6.1 (BST)

Commit message: added sd card, dividers, and connector
Parts:
- added C1: 10uF, Adafruit SDIO microSD:0805-NO, symbol Adafruit SDIO microSD-eagle-import:microbuilder_CAP_CERAMIC0805-NOOUTLINE
- added C2: 0.1uF, Adafruit SDIO microSD:0603-NO, symbol Adafruit SDIO microSD-eagle-import:microbuilder_CAP_CERAMIC0603_NO
- added J3: Conn_01x04, symbol Connector_Generic:Conn_01x04
- added JP1: HEADER-1X970MIL, Adafruit SDIO microSD:1X09_ROUND_70, symbol Adafruit SDIO microSD-eagle-import:microbuilder_HEADER-1X970MIL
- added R1: 114k, symbol Device:R
- added R2, R4: 57k, symbol Device:R
- added R3: 300k, symbol Device:R
- added R5: 303k, symbol Device:R
- added R6: 198k, symbol Device:R
- added R7, R8: 47K, Adafruit SDIO microSD:RESPACK_4X0603, symbol Adafruit SDIO microSD-eagle-import:microbuilder_RESISTOR_4PACK
- added X1: microSD, Adafruit SDIO microSD:MICROSD, symbol Adafruit SDIO microSD-eagle-import:microbuilder_MICROSD
Connections:
- net GND: now also C1.2, C2.2, JP1.2, R2.2, R4.2, R6.2, X1.6 (GND@3), X1.MT1 (GND@2), X1.MT2 (GND@1)
- net VP_PIN: now reaches J5.3 (Pin_3), U2.3 (SENSOR_VP)
- net VP_PIN: now also R1.2, R2.1
- net VN_PIN: now reaches J5.4 (Pin_4), U2.4 (SENSOR_VN)
- net VN_PIN: now also R3.2, R4.1
- net 35_PIN: now reaches J3.4 (Pin_4), U2.35 (TXD0)
- net 35_PIN: now also R5.2, R6.1
- new net: J3.2 (Pin_2), R3.1
- new net: J3.1 (Pin_1), R1.1
- new net: J3.3 (Pin_3), R5.1
- new net 3.3V: C1.1, C2.1, JP1.1, R7.1, R7.2 (1), R7.3 (1), R8.1, R8.2 (1), R8.3 (1), R8.4 (1), X1.4 (SD_VDD)
- new net CARDDET: JP1.9, R7.8 (2), X1.CD1 (CARD_DETECT)
- new net CS: JP1.6, R8.7 (2), X1.2 (CS)
- new net DAT1: JP1.7, R7.7 (2), X1.8 (DAT1)
- new net DAT2: JP1.8, R8.8 (2), X1.1 (DAT2)
- new net DI: JP1.5, R8.6 (2), X1.3 (DATA_IN)
- new net DO: JP1.4, R7.6 (2), X1.7 (DATA_OUT)
- new net SCLK: JP1.3, R8.5 (2), X1.5 (SCLK)

Commit message: updated schematic to match diagram
Parts:
- removed J3: Conn_01x04, symbol Connector_Generic:Conn_01x04
- added J6: Conn_01x03, symbol Connector_Generic:Conn_01x03
- added J7: Conn_01x06, symbol Connector_Generic:Conn_01x06
- C1: footprint Adafruit SDIO microSD:0805-NO -> Capacitor_SMD:C_0805_2012Metric
- C2: footprint Adafruit SDIO microSD:0603-NO -> Capacitor_SMD:C_0805_2012Metric
- J1: renamed from J2; footprint (none) -> Connector_PinHeader_2.54mm:PinHeader_1x04_P2.54mm_Vertical
- R1: renamed from R8; footprint Adafruit SDIO microSD:RESPACK_4X0603 -> Resistor_SMD:R_0815_2038Metric
- R1: renamed from R7; footprint Adafruit SDIO microSD:RESPACK_4X0603 -> Resistor_SMD:R_0815_2038Metric
- R10: renamed from R5; value 303k -> 100k; footprint (none) -> Resistor_SMD:R_0805_2012Metric
- R2: renamed from R8; footprint Adafruit SDIO microSD:RESPACK_4X0603 -> Resistor_SMD:R_0805_2012Metric
- R2: renamed from R7; footprint Adafruit SDIO microSD:RESPACK_4X0603 -> Resistor_SMD:R_0805_2012Metric
- R5: renamed from R2; value 57k -> 100k; footprint (none) -> Resistor_SMD:R_0805_2012Metric
- R6: renamed from R4; value 57k -> 100k; footprint (none) -> Resistor_SMD:R_0805_2012Metric
- R7: renamed from R6; value 198k -> 100k; footprint (none) -> Resistor_SMD:R_0805_2012Metric
- R8: renamed from R1; value 114k -> 200k; footprint (none) -> Resistor_SMD:R_0805_2012Metric
- R9: renamed from R3; value 300k -> 200k; footprint (none) -> Resistor_SMD:R_0805_2012Metric
- renumbered C5 to C3, C6 to C5, C7 to C6, C1 to C7, C2 to C8, C3 to C9, J5 to J2, J1 to J5, R4 to R11, R2 to R12, R3 to R13, R5 to R3, R6 to R4, U6 to U1, U5 to U3, U3 to U5
Connections:
- net 35_PIN: no longer R10.2, R7.1
- net BUCK_5V: now also J6.1 (Pin_1)
- net GND: now also J6.3 (Pin_3), J7.1 (Pin_1), J7.4 (Pin_4)
- net at R9.1: now also J7.5 (Pin_5)
- net at R8.1: now also J7.3 (Pin_3), J7.6 (Pin_6)
- net at R10.1: now also J7.2 (Pin_2)
- new net: R10.2, R7.1
Other:
- moved on the sheet: R10, R5, R6, R7, R8, R9

Commit message: schematic done before layout
Parts:
- Brake1: renamed from J6; footprint (none) -> TerminalBlock_Phoenix:TerminalBlock_Phoenix_MKDS-1,5-3-5.08_1x03_P5.08mm_Horizontal
- J2, J3: footprint (none) -> Connector_PinSocket_2.54mm:PinSocket_1x19_P2.54mm_Vertical
- J4: renamed from J5; footprint (none) -> Connector_PinSocket_2.54mm:PinSocket_1x02_P2.54mm_Vertical
- L1: footprint PROVE:WE-LQS_5040 -> Capacitor_SMD:C_1206_3216Metric_Pad1.33x1.80mm_HandSolder
- Pedal1: renamed from J7; footprint (none) -> TerminalBlock_Phoenix:TerminalBlock_Phoenix_MKDS-1,5-6_1x06_P5.00mm_Horizontal
- renumbered R9 to R10, R7 to R5, R5 to R6, R6 to R7, R10 to R8, R8 to R9
Connections:
- net 35_PIN: now also R5.1, R8.2
- net BUCK_5V: now also Pedal1.3 (Pin_3), Pedal1.6 (Pin_6), R9.1
- net VN_PIN: now also Pedal1.5 (Pin_5), R10.1
- net 34_PIN: now reaches Brake1.2 (Pin_2)
- net 34_PIN: now also J3.5 (Pin_5), U2.34 (RXD0)
Other:
- moved on the sheet: Brake1, Pedal1, R10, R5, R6, R7, R8, R9
