File: TELEM/Microcontroller.kicad_sch (KiCad schematic)
At the start: 16 parts, among them J1 Conn_01x02, J4 Conn_01x02_Pin, M3 MountingHole, M3_ MountingHole, U2 ESP32-DEVKIT-C, U6 TJA1050T/CM,118

Commit message: made updates to the buck to better adhere to TIs layout guidelines. Updated buck to output 5.2V instead of 5.3V, since new Ebyte datasheet revision now suggests 5 to 5.25V, as opposed to the previous 5 to 5.5V. Updated the MCU PCB with the new buck, as well as the connectors. added two additional gpio pins broken out of MCU PCB for probable, but unspecified future use.
Parts:
- removed J1: Conn_01x02, PROVE-footprints:TE_1877285-2, symbol Connector_Generic:Conn_01x02
- added C3, C4: 47uF, Capacitor_Tantalum_SMD:CP_EIA-3528-21_Kemet-B_HandSolder, symbol 10TPE47MAZB:10TPE47MAZB
- renumbered Cout2 to C2, M3_ to M3_1, R6 to R1, U6 to U3
Connections:
- net GND: now also C3.2, C4.2
- net 5.3V OUT renamed 5.2V_OUT
- net 5.2V_OUT: now also C3.1, C4.1
Other:
- sheet 25_To_5p3V_step_down renamed 25_to_5p2V_step_down
- sheet 25_to_5p2V_step_down: file 5V_Buck.kicad_sch -> ../buck_converter.kicad_blocks/25_to_5p2V_step_down.kicad_block/25_to_5p2V_step_down.kicad_sch
- sheet 25_to_5p2V_step_down ports: added 5.2V_Out; removed 5.3V_Out
- moved on the sheet: M3
