File: buck_converter.kicad_blocks/25_to_5p2V_step_down.kicad_block/25_to_5p2V_step_down.kicad_sch (KiCad schematic)
At the start: 12 parts, among them U7 TPS54560BQDDARQ1

Commit message: made updates to the buck to better adhere to TIs layout guidelines. Updated buck to output 5.2V instead of 5.3V, since new Ebyte datasheet revision now suggests 5 to 5.25V, as opposed to the previous 5 to 5.5V. Updated the MCU PCB with the new buck, as well as the connectors. added two additional gpio pins broken out of MCU PCB for probable, but unspecified future use.
Parts:
- added Cin1: 47uF, Capacitor_SMD:CP_Elec_6.3x7.7, symbol Device:C_Polarized_US
- added J3: Conn_01x02, PROVE-footprints:TE_1877285-2, symbol Connector_Generic:Conn_01x02
- Rfbb1: value 11kOhm -> 11.8kOhm; Purchase Link https://www.mouser.com/en/ProductDetail/Vishay/CRCW120611K0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 -> https://www.mouser.com/en/ProductDetail/Vishay/CRCW120611K8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; Specs Resistance: 11 kΩ Tolerance: 1.0% Power: 250 mW -> Resistance: 11.8 kΩ Tolerance: 1% Power: 250 mW
- Rfbt1: value 61.9kOhm -> 64.9kOhm; Purchase Link https://www.mouser.com/en/ProductDetail/Vishay/CRCW120661K9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 -> https://www.mouser.com/en/ProductDetail/Vishay/CRCW120664K9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; Specs Resistance: 61.9 kΩ Tolerance: 1.0% Power: 250 mW -> Resistance: 64.9 kΩ Tolerance: 1.0% Power: 250 mW
- renumbered Cin1 to Cin2, U7 to U4
Connections:
- net GND: now also Cin1.2, J3.2 (Pin_2)
- net 25V_In: no longer names the net of Cin2.2, U4.2 (VIN)
- net 25V_In: now also Cin1.1, J3.1 (Pin_1)
- net 5.3V_Out renamed 5.2V_Out
Other:
- moved on the sheet: Cin2

Commit message: updated Julias IMU to use the revised buck converter and connectors. made the back plane mostly a ground plane (for the buck converter)
Parts:
- renumbered J3 to J1, U4 to U1
Changed lines of the file:
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@@
 		(dnp no)
 		(fields_autoplaced yes)
-		(property "Reference" "U4"
+		(property "Reference" "U1"
 			(at 125.73 54.61 0)
 			(show_name no)
@@
 			(project "MCU"
 				(path "/c58806c5-432f-4c41-8983-8e5fd30a3703/17ad73fb-67eb-456b-8672-13a62eb66df9"
-					(reference "U4")
+					(reference "U1")
 					(unit 1)
 				)
@@
 		(dnp no)
 		(fields_autoplaced yes)
-		(property "Reference" "J3"
+		(property "Reference" "J1"
 			(at 26.67 66.04 0)
 			(hide yes)
@@
 			(project "MCU"
 				(path "/c58806c5-432f-4c41-8983-8e5fd30a3703/17ad73fb-67eb-456b-8672-13a62eb66df9"
-					(reference "J3")
+					(reference "J1")
 					(unit 1)
 				)
@@
 		)
 	)
-	(sheet_instances
-		(path "/"
-			(page "1")
-		)
-	)
