File: PDB/buck_to_20V.kicad_sch (KiCad schematic)
At the start: 14 parts, among them J1 Conn_01x02, U1 TPS54560BQDDARQ1

Commit message: PDB_Schematic mostly updated
Parts:
- removed J1: Conn_01x02, PROVE-footprints:TE_1877285-2, symbol Connector_Generic:Conn_01x02
- renumbered Cboot1 to Cboot2, Ccmp1 to Ccmp5, Ccmp2 to Ccmp6, Cin1 to Cin3, Cin2 to Cin4, Cout1 to Cout4, D1 to D3, L1 to L2, RCmp1 to RCmp2, Rfbb1 to Rfbb2, Rfbt1 to Rfbt2, Rt1 to Rt2, U1 to U16
Connections:
- net 25V_In: now reaches Cin3.1, Cin4.2, U16.2 (VIN)
- net 5.2V_Out renamed 20V_Out
Other:
- moved on the sheet: Cboot2, Ccmp5, Ccmp6, Cin3, Cin4, Cout4, D3, L2, RCmp2, Rfbb2, Rfbt2, Rt2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
