File: PDB/buck_to_20V.kicad_sch (KiCad schematic)
At the start: 17 parts, among them U16 TPS54560BQDDARQ1

Commit message: updates to 12V, PDB, and IMU (leave me alone)
Other:
- moved on the sheet: C21, C22, Cboot2, Cin3, Cin4, Cout2, Cout3, Cout4, D3, L2, R1, R2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
