File: PDB/buck_to_5V.kicad_sch (KiCad schematic)
At the start: 14 parts, among them J1 Conn_01x02, U1 TPS54560BQDDARQ1

Commit message: PDB_Schematic mostly updated
Parts:
- removed J1: Conn_01x02, PROVE-footprints:TE_1877285-2, symbol Connector_Generic:Conn_01x02
- removed U1: TPS54560BQDDARQ1, Package_SO:SOIC-8-1EP_3.9x4.9mm_P1.27mm_EP2.29x3mm, symbol TPS54560BQDDARQ1:TPS54560BQDDARQ1
- added U4: TPS54560BQDDARQ1, Package_SO:SOIC-8-1EP_3.9x4.9mm_P1.27mm_EP2.29x3mm, symbol TPS54560BQDDARQ1:TPS54560BQDDARQ1
Connections:
- net GND: now also U4.7 (GND), U4.9 (EPAD)
- net 25V_IN: now reaches Cin1.1, Cin2.2
- net 25V_IN: now also U4.2 (VIN)
- net at Cboot1.1, D1.1, L1.2: now also U4.8 (SW)
- net at Cboot1.2: now also U4.1 (BOOT)
- net at Rt1.2: now also U4.4 (RT/CLK)
- net at Rfbb1.1, Rfbt1.1: now also U4.5 (FB)
- net at Ccmp2.1, RCmp1.2: now also U4.6 (COMP)
