File: IMU_PCB/Microcontroller.kicad_pcb (KiCad board)
At the start: 2 copper layers, 100 x 59.2 mm, 32 parts, among them IC1 TJA1044BT/0Z, J2 39-28-1023, J25 39-28-1023, U15 LM4040CELT-3.0, U2 ESP32-DEVKIT-C, U4 TPS54560BQDDARQ1, U7 SparkFun: ISM330DHCX, MMC5983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, U8 SDIO Card Breakout Board, U9 AM2302

Commit message: updates to 12V, PDB, and IMU (leave me alone)
Changed lines of the file:
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@@
+	)
+	(segment
+		(start 129.56 67.3025)
+		(end 131.5875 67.3025)
+		(width 1)
+		(layer "F.Cu")
+		(net "Net-(U15-K)")
+	)
+	(segment
+		(start 130.19 64.98)
+		(end 129.3975 64.98)
+		(width 1)
+		(layer "F.Cu")
+		(net "Net-(U15-K)")
+	)
+	(segment
+		(start 131.83 66.62)
+		(end 130.19 64.98)
+		(width 1)
+		(layer "F.Cu")
+		(net "Net-(U15-K)")
+	)
+	(segment
+		(start 172.9125 103.9275)
+		(end 172.81 103.9275)
+		(width 0.2)
+		(layer "F.Cu")
+		(net "Net-(U15-K)")
+	)
+	(segment
+		(start 133.1 66.62)
+		(end 131.83 66.62)
+		(width 1)
+		(layer "F.Cu")
+		(net "Net-(U15-K)")
+	)
+	(segment
+		(start 129.56 66.17)
+		(end 129.56 67.3025)
+		(width 1)
+		(layer "F.Cu")
+		(net "Net-(U15-K)")
+	)
+	(segment
+		(start 129.3975 66.0075)
+		(end 129.56 66.17)
+		(width 1)
+		(layer "F.Cu")
+		(net "Net-(U15-K)")
+	)
+	(segment
+		(start 132.74 66.98)
+		(end 133.1 66.62)
+		(width 1)
+		(layer "F.Cu")
+		(net "Net-(U15-K)")
+	)
+	(segment
+		(start 129.3975 64.98)
+		(end 129.3975 66.0075)
+		(width 1)
+		(layer "F.Cu")
+		(net "Net-(U15-K)")
+	)
+	(segment
+		(start 131.91 66.98)
+		(end 132.74 66.98)
+		(width 1)
+		(layer "F.Cu")
+		(net "Net-(U15-K)")
+	)
+	(segment
+		(start 173.7 103.14)
+		(end 172.9125 103.9275)
+		(width 0.2)
+		(layer "F.Cu")
+		(net "Net-(U15-K)")
+	)
+	(segment
+		(start 131.5875 67.3025)
+		(end 131.91 66.98)
+		(width 1)
+		(layer "F.Cu")
+		(net "Net-(U15-K)")
+	)
+	(segment
+		(start 175.2 103.14)
+		(end 173.7 103.14)
+		(width 0.2)
+		(layer "F.Cu")
+		(net "Net-(U15-K)")
+	)
+	(via
+		(at 175.2 103.14)
+		(size 0.6)
+		(drill 0.3)
+		(layers "F.Cu" "B.Cu")
+		(net "Net-(U15-K)")
+	)
+	(segment
+		(start 198.26 63.99)
+		(end 198.26 75.65)
+		(width 0.3)
+		(layer "B.Cu")
+		(net "Net-(U15-K)")
+	)
+	(segment
+		(start 182.35 93.97)
+		(end 182.35 96.41)
+		(width 0.3)
+		(layer "B.Cu")
+		(net "Net-(U15-K)")
+	)
+	(segment
+		(start 175.62 103.14)
+		(end 182.35 96.41)
+		(width 0.2)
+		(layer "B.Cu")
+		(net "Net-(U15-K)")
+	)
+	(segment
+		(start 175.2 103.14)
+		(end 175.62 103.14)
+		(width 0.2)
+		(layer "B.Cu")
+		(net "Net-(U15-K)")
+	)
+	(segment
+		(start 135.4 66.62)
+		(end 148.77 53.25)
+		(width 0.3)
+		(layer "B.Cu")
+		(net "Net-(U15-K)")
+	)
+	(segment
+		(start 195.8 80.52)
+		(end 182.35 93.97)
+		(width 0.3)
+		(layer "B.Cu")
+		(net "Net-(U15-K)")
+	)
+	(segment
+		(start 198.26 75.65)
+		(end 195.8 78.11)
+		(width 0.3)
+		(layer "B.Cu")
+		(net "Net-(U15-K)")
+	)
+	(segment
+		(start 187.52 53.25)
+		(end 198.26 63.99)
+		(width 0.3)
+		(layer "B.Cu")
+		(net "Net-(U15-K)")
+	)
+	(segment
+		(start 148.77 53.25)
+		(end 187.52 53.25)
+		(width 0.3)
+		(layer "B.Cu")
+		(net "Net-(U15-K)")
+	)
+	(segment
+		(start 133.1 66.62)
+		(end 135.4 66.62)
+		(width 0.3)
+		(layer "B.Cu")
+		(net "Net-(U15-K)")
+	)
+	(segment
+		(start 195.8 78.11)
+		(end 195.8 80.52)
+		(width 0.3)
+		(layer "B.Cu")
+		(net "Net-(U15-K)")
 	)
 	(segment
@@
 	)
 	(segment
-		(start 159.5895 71.7)
+		(start 158.5 71.7)
+		(end 159.41 71.7)
+		(width 0.2)
+		(layer "F.Cu")
+		(net "Net-(U2-IO21)")
+	)
+	(segment
+		(start 164.4685 66.6415)
 		(end 164.648 66.6415)
 		(width 0.2)
@@
 	)
 	(segment
-		(start 158.5 71.7)
-		(end 159.5895 71.7)
+		(start 162.4385 66.8615)
+		(end 163.708 66.8615)
+		(width 0.2)
+		(layer "F.Cu")
+		(net "Net-(U2-IO21)")
+	)
+	(segment
+		(start 161.02 70.09)
+		(end 161.02 68.28)
+		(width 0.2)
+		(layer "F.Cu")
+		(net "Net-(U2-IO21)")
+	)
+	(segment
+		(start 161.02 68.28)
+		(end 162.4385 66.8615)
+		(width 0.2)
+		(layer "F.Cu")
+		(net "Net-(U2-IO21)")
+	)
+	(segment
+		(start 159.41 71.7)
+		(end 161.02 70.09)
 		(width 0.2)
 		(layer "F.Cu")
@@
 		(net "Net-(C24-Pad2)")
 	)
-	(segment
-		(start 129.56 67.3025)
-		(end 131.5875 67.3025)
-		(width 1)
-		(layer "F.Cu")
-		(net "Net-(U15-K)")
-	)
-	(segment
-		(start 130.19 64.98)
-		(end 129.3975 64.98)
-		(width 1)
-		(layer "F.Cu")
-		(net "Net-(U15-K)")
-	)
-	(segment
-		(start 131.83 66.62)
-		(end 130.19 64.98)
-		(width 1)
-		(layer "F.Cu")
-		(net "Net-(U15-K)")
-	)
-	(segment
-		(start 172.9125 103.9275)
-		(end 172.81 103.9275)
-		(width 0.2)
-		(layer "F.Cu")
-		(net "Net-(U15-K)")
-	)
-	(segment
-		(start 133.1 66.62)
-		(end 131.83 66.62)
-		(width 1)
-		(layer "F.Cu")
-		(net "Net-(U15-K)")
-	)
-	(segment
-		(start 129.56 66.17)
-		(end 129.56 67.3025)
-		(width 1)
-		(layer "F.Cu")
-		(net "Net-(U15-K)")
-	)
-	(segment
-		(start 129.3975 66.0075)
-		(end 129.56 66.17)
-		(width 1)
-		(layer "F.Cu")
-		(net "Net-(U15-K)")
-	)
-	(segment
-		(start 132.74 66.98)
-		(end 133.1 66.62)
-		(width 1)
-		(layer "F.Cu")
-		(net "Net-(U15-K)")
-	)
-	(segment
-		(start 129.3975 64.98)
-		(end 129.3975 66.0075)
-		(width 1)
-		(layer "F.Cu")
-		(net "Net-(U15-K)")
-	)
-	(segment
-		(start 131.91 66.98)
-		(end 132.74 66.98)
-		(width 1)
-		(layer "F.Cu")
-		(net "Net-(U15-K)")
-	)
-	(segment
-		(start 173.7 103.14)
-		(end 172.9125 103.9275)
-		(width 0.2)
-		(layer "F.Cu")
-		(net "Net-(U15-K)")
-	)
-	(segment
-		(start 131.5875 67.3025)
-		(end 131.91 66.98)
-		(width 1)
-		(layer "F.Cu")
-		(net "Net-(U15-K)")
-	)
-	(segment
-		(start 175.2 103.14)
-		(end 173.7 103.14)
-		(width 0.2)
-		(layer "F.Cu")
-		(net "Net-(U15-K)")
-	)
-	(via
-		(at 175.2 103.14)
-		(size 0.6)
-		(drill 0.3)
-		(layers "F.Cu" "B.Cu")
-		(net "Net-(U15-K)")
-	)
-	(segment
-		(start 198.26 63.99)
-		(end 198.26 75.65)
-		(width 0.3)
-		(layer "B.Cu")
-		(net "Net-(U15-K)")
-	)
-	(segment
-		(start 182.35 93.97)
-		(end 182.35 96.41)
-		(width 0.3)
-		(layer "B.Cu")
-		(net "Net-(U15-K)")
-	)
-	(segment
-		(start 175.62 103.14)
-		(end 182.35 96.41)
-		(width 0.2)
-		(layer "B.Cu")
-		(net "Net-(U15-K)")
-	)
-	(segment
-		(start 175.2 103.14)
-		(end 175.62 103.14)
-		(width 0.2)
-		(layer "B.Cu")
-		(net "Net-(U15-K)")
-	)
-	(segment
-		(start 135.4 66.62)
-		(end 148.77 53.25)
-		(width 0.3)
-		(layer "B.Cu")
-		(net "Net-(U15-K)")
-	)
-	(segment
-		(start 195.8 80.52)
-		(end 182.35 93.97)
-		(width 0.3)
-		(layer "B.Cu")
-		(net "Net-(U15-K)")
-	)
-	(segment
-		(start 198.26 75.65)
-		(end 195.8 78.11)
-		(width 0.3)
-		(layer "B.Cu")
-		(net "Net-(U15-K)")
-	)
-	(segment
-		(start 187.52 53.25)
-		(end 198.26 63.99)
-		(width 0.3)
-		(layer "B.Cu")
-		(net "Net-(U15-K)")
-	)
-	(segment
-		(start 148.77 53.25)
-		(end 187.52 53.25)
-		(width 0.3)
-		(layer "B.Cu")
-		(net "Net-(U15-K)")
-	)
-	(segment
-		(start 133.1 66.62)
-		(end 135.4 66.62)
-		(width 0.3)
-		(layer "B.Cu")
-		(net "Net-(U15-K)")
-	)
-	(segment
-		(start 195.8 78.11)
-		(end 195.8 80.52)
-		(width 0.3)
-		(layer "B.Cu")
-		(net "Net-(U15-K)")
-	)
 	(zone
